File: FaderCtrl/HW/PCB/FaderCtrl/FaderCtrl.kicad_sch (KiCad schematic)
At the start: 89 parts, among them J1 PDI, J2 Barrel_Jack_MountingPin, J3 PWM, J4 PORTD, J5 MPS, J6 MPP, J7 MPN, P1 USB_C_Plug_USB2.0, U1 ATxmega256A3BU-A, U2 TSR_1-2450, U3 AMS1117-3.3, Y1 32k

Commit message: a
Parts:
- removed J4: PORTD, symbol Connector_Generic:Conn_01x10
- added C13, C17, C22: 10n, Capacitor_SMD:C_0603_1608Metric_Pad1.08x0.95mm_HandSolder, symbol Device:C
- added C2, C4: 10p, Capacitor_SMD:C_0603_1608Metric_Pad1.08x0.95mm_HandSolder, symbol Device:C
- added J1: UART, Connector_PinSocket_2.54mm:PinSocket_1x03_P2.54mm_Vertical, symbol Connector_Generic:Conn_01x03
- added J3: PORTE, Connector_PinSocket_1.27mm:PinSocket_1x08_P1.27mm_Vertical, symbol Connector_Generic:Conn_01x08
- added J4: VBAT, Connector_PinSocket_2.54mm:PinSocket_1x02_P2.54mm_Vertical, symbol Connector_Generic:Conn_01x02
- added R2: 56k, Resistor_SMD:R_0603_1608Metric_Pad0.98x0.95mm_HandSolder, symbol Device:R
- added R3: 5k1, Resistor_SMD:R_0603_1608Metric_Pad0.98x0.95mm_HandSolder, symbol Device:R
- added SW1: BTN1, footprints:SW_PUSH_6mm_2pins, symbol Switch:SW_Push
- added SW2: BTN2, footprints:SW_PUSH_6mm_2pins, symbol Switch:SW_Push
- added SW3: BTN3, footprints:SW_PUSH_6mm_2pins, symbol Switch:SW_Push
- added TP2: Vconn, TestPoint:TestPoint_Pad_D1.0mm, symbol Connector:TestPoint
- added TP3: TR1, TestPoint:TestPoint_THTPad_D1.0mm_Drill0.5mm, symbol Connector:TestPoint
- added TP4: ~{OE}, TestPoint:TestPoint_Pad_D1.0mm, symbol Connector:TestPoint
- added TP5: SLED1, TestPoint:TestPoint_Pad_D1.0mm, symbol Connector:TestPoint
- added TP8: SL1, TestPoint:TestPoint_THTPad_D1.0mm_Drill0.5mm, symbol Connector:TestPoint
- added Y2: 12M, Crystal:Crystal_SMD_HC49-SD, symbol Device:Crystal
- C1: now not fitted
- C3: renamed from C2; now not fitted
- D3: renamed from D2; footprint (none) -> LED_SMD:LED_Cree-PLCC4_3.2x2.8mm_CCW
- D5: renamed from D3; footprint (none) -> LED_SMD:LED_Cree-PLCC4_3.2x2.8mm_CCW
- J6: renamed from J3; footprint (none) -> Connector_PinSocket_1.27mm:PinSocket_1x09_P1.27mm_Vertical
- J7: renamed from J5; footprint (none) -> Connector_PinSocket_2.54mm:PinSocket_1x04_P2.54mm_Vertical
- J8: renamed from J6; footprint (none) -> Connector_PinSocket_2.54mm:PinSocket_1x04_P2.54mm_Vertical
- J9: renamed from J7; footprint (none) -> Connector_PinSocket_2.54mm:PinSocket_1x04_P2.54mm_Vertical
- JP1: value Jumper_3_Bridged12 -> Vin3v3
- JP2: value Jumper_2_Small_Bridged -> VDDA
- MP1, MP2, MP3, MP4: footprint Connector_PinSocket_2.54mm:PinSocket_1x09_P2.54mm_Vertical -> Connector_PinSocket_2.54mm:PinSocket_1x10_P2.54mm_Vertical
- NT1: value NetTie_2 -> GNDD
- NT2: value NetTie_2 -> GNDA
- TP9: renamed from TP4; footprint (none) -> TestPoint:TestPoint_THTPad_D1.0mm_Drill0.5mm
- U4, U5: footprint HTSSOP-20-1EP_4.4x6.5mm_P0.65mm_EP3.4x6.5mm -> Package_SO:HTSSOP-20-1EP_4.4x6.5mm_P0.65mm_EP3.4x6.5mm
- Y1: symbol Device:Crystal_GND2 -> Device:Crystal_GND3; now not fitted
- renumbered C8 to C10, C9 to C11, C10 to C12, C11 to C14, C12 to C15, C13 to C16, C14 to C18, C16 to C19, C19 to C20, C15 to C21, C17 to C23, C18 to C24, C20 to C25, C21 to C26, C22 to C27, C23 to C28, C24 to C29, C25 to C30, C26 to C31, C27 to C32, C28 to C33, C29 to C34, C30 to C35, C31 to C36, C32 to C37, C33 to C38, C34 to C39, C35 to C40, C36 to C41, C37 to C42, C38 to C43, C39 to C44, C3 to C5, C4 to C6, C5 to C7, C6 to C8, C7 to C9, D4 to D2, D5 to D4, J1 to J2, J2 to J5, R6 to R10, R7 to R11, R10 to R12, R11 to R13, R8 to R6, R9 to R7, R2 to R8, R3 to R9, TP5 to TP10, TP6 to TP11, TP2 to TP6, TP3 to TP7
Connections:
- net BTN0 is gone; now on net BTN1: U1.11 (PB5)
- net PD0 is gone; now on net SLED1: U1.26 (PD0)
- net PD1 is gone; now on net SLED2: U1.27 (PD1)
- net PD2 is gone; now on net SLED3: U1.28 (PD2)
- net PD3 is gone; now on net SLED4: U1.29 (PD3)
- net PD4 is gone; now on net CP: U1.30 (PD4)
- net PD5 is gone; now on net ~{CP}: U1.31 (PD5)
- net PD6 is gone; now on net D-: U1.32 (PD6)
- net PD7 is gone; now on net D+: U1.33 (PD7)
- net +5V: no longer D2.1
- net BTN1: now also C13.1, SW1.2; no longer U1.12 (PB6)
- net BTN2: now also U1.12 (PB6), C17.1, SW2.2; no longer U1.13 (PB7)
- net CP: no longer U1.40 (PE4)
- net GNDD: now also Y1.3, C13.2, C17.2, C2.2, C22.2, C4.2, J1.3 (Pin_3), J3.8 (Pin_8), J4.2 (Pin_2), R3.1, SW1.1, SW2.1, SW3.1; no longer Y1.2
- net SL1: now also TP8.1
- net SLED1: now also TP5.1; no longer U1.36 (PE0)
- net SLED2: no longer U1.37 (PE1)
- net SLED3: no longer U1.38 (PE2)
- net SLED4: no longer U1.39 (PE3)
- net TP3: now also U1.50 (PF4); no longer U1.48 (PF2)
- net TP4: now also U1.54 (PF6); no longer U1.49 (PF3)
- net TR1: now also TP3.1
- net VBUS: now also R2.2
- net VDD: now also J3.1 (Pin_1)
- net Vdrive: now also D2.1
- net XTAL1: now also C2.1, Y2.1; no longer C3.1, Y1.3
- net XTAL2: now also C4.1, Y2.2; no longer C1.1, Y1.1
- net ~{CP}: no longer U1.41 (PE5)
- net ~{OE}: now also TP4.1
- net TOSC2: now reaches U1.42 (TOSC2)
- net TOSC2: now also C3.1, Y1.1
- net TOSC1: now reaches U1.43 (TOSC1)
- net TOSC1: now also C1.1, Y1.2
- net Vbat: now reaches U1.51 (VBAT)
- net Vbat: now also J4.1 (Pin_1)
- net CC: now reaches P1.A5 (CC)
- net CC: now also R2.1, R3.2
- net D+: now reaches P1.A6 (D+)
- net D-: now reaches P1.A7 (D-)
- net at P1.B5 (VCONN): now also TP2.1
- new net: J3.2 (Pin_2), U1.36 (PE0)
- new net: J3.3 (Pin_3), U1.37 (PE1)
- new net: J3.4 (Pin_4), U1.38 (PE2)
- new net: J3.5 (Pin_5), U1.39 (PE3)
- new net: J3.6 (Pin_6), U1.40 (PE4)
- new net: J3.7 (Pin_7), U1.41 (PE5)
- new net BTN3: C22.1, SW3.2, U1.13 (PB7)
- new net RXD: J1.1 (Pin_1), U1.48 (PF2)
- new net TXD: J1.2 (Pin_2), U1.49 (PF3)
- no-connect marks 4 -> 3
Other:
- company: (none) -> Xavier Bourlot
- title: (none) -> Fader Controller
- moved on the sheet: C42, C43, D3, D5, MP1D, MP2D, MP3D, MP4D, NT1, NT2, P1, R10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

Commit message: a
Parts:
- added C45, C46: 100n, Capacitor_SMD:C_0603_1608Metric_Pad1.08x0.95mm_HandSolder, symbol Device:C
Connections:
- net BTN1: now also U1.7 (PB1); no longer U1.11 (PB5)
- net BTN2: now also U1.8 (PB2); no longer U1.12 (PB6)
- net BTN3: now also U1.9 (PB3); no longer U1.13 (PB7)
- net GNDA: now also C45.2, C46.2
- net LED0: now also U1.2 (PA4); no longer U1.6 (AREF/PB0)
- net LED1: now also U1.3 (PA5); no longer U1.7 (PB1)
- net LED2: now also U1.4 (PA6); no longer U1.8 (PB2)
- net LED3: now also U1.5 (PA7); no longer U1.9 (PB3)
- net SL1: now also U1.10 (PB4); no longer U1.2 (PA4)
- net SL2: now also U1.11 (PB5); no longer U1.3 (PA5)
- net SL3: now also U1.12 (PB6); no longer U1.4 (PA6)
- net SL4: now also U1.13 (PB7); no longer U1.5 (PA7)
- net VDDA: now also U1.6 (AREF/PB0), C45.1, C46.1
- net ~{OE}: now also U1.55 (PF7); no longer U1.10 (PB4)
- no-connect marks 3 -> 2
Other:
- moved on the sheet: TP4, TP8

Commit message: a
Parts:
- removed J7: MPS, Connector_PinSocket_2.54mm:PinSocket_1x04_P2.54mm_Vertical, symbol Connector_Generic:Conn_01x04
- removed J8: MPP, Connector_PinSocket_2.54mm:PinSocket_1x04_P2.54mm_Vertical, symbol Connector_Generic:Conn_01x04
- removed J9: MPN, Connector_PinSocket_2.54mm:PinSocket_1x04_P2.54mm_Vertical, symbol Connector_Generic:Conn_01x04
- added J10: MP4, Connector_PinHeader_2.54mm:PinHeader_1x03_P2.54mm_Vertical, symbol Connector_Generic:Conn_01x03
- added J7: MP1, Connector_PinHeader_2.54mm:PinHeader_1x03_P2.54mm_Vertical, symbol Connector_Generic:Conn_01x03
- added J8: MP2, Connector_PinHeader_2.54mm:PinHeader_1x03_P2.54mm_Vertical, symbol Connector_Generic:Conn_01x03
- added J9: MP3, Connector_PinHeader_2.54mm:PinHeader_1x03_P2.54mm_Vertical, symbol Connector_Generic:Conn_01x03
- MP1, MP2, MP3, MP4: footprint Connector_PinSocket_2.54mm:PinSocket_1x10_P2.54mm_Vertical -> footprints:PSM01-082A-103B2_MotorizedPot
- U4, U5: footprint Package_SO:HTSSOP-20-1EP_4.4x6.5mm_P0.65mm_EP3.4x6.5mm -> HTSSOP-20-1EP_4.4x6.5mm_P0.65mm_EP3.4x6.5mm
Connections:
- net GND: now also U4.21 (EP), U5.21 (EP)
- net GNDA: now also MP1.9 (3'), MP2.9 (3'), MP3.9 (3'), MP4.9 (3'); no longer MP1.10 (3'), MP2.10 (3'), MP3.10 (3'), MP4.10 (3')
- net MP1N: now also MP4.5 (1), J7.3 (Pin_3); no longer MP4.6 (1)
- net MP1P: now also MP4.3, J7.1 (Pin_1); no longer MP4.4 (3)
- net MP1S: now also MP4.4 (2), J7.2 (Pin_2); no longer MP4.5 (2)
- net MP2N: now also MP3.5 (1), J8.3 (Pin_3); no longer MP3.6 (1)
- net MP2P: now also MP3.3, J8.1 (Pin_1); no longer MP3.4 (3)
- net MP2S: now also MP3.4 (2), J8.2 (Pin_2); no longer MP3.5 (2)
- net MP3N: now also MP2.5 (1), J9.3 (Pin_3); no longer MP2.6 (1)
- net MP3P: now also MP2.3, J9.1 (Pin_1); no longer MP2.4 (3)
- net MP3S: now also MP2.4 (2), J9.2 (Pin_2); no longer MP2.5 (2)
- net MP4N: now also MP1.5 (1), J10.3 (Pin_3); no longer MP1.6 (1)
- net MP4P: now also MP1.3, J10.1 (Pin_1); no longer MP1.4 (3)
- net MP4S: now also MP1.4 (2), J10.2 (Pin_2); no longer MP1.5 (2)
- net TP1: now also MP1.6 (T); no longer MP1.7 (T)
- net TP2: now also MP2.6 (T); no longer MP2.7 (T)
- net TP3: now also MP3.6 (T); no longer MP3.7 (T)
- net TP4: now also MP4.6 (T); no longer MP4.7 (T)
- net TR1: now also MP1.8 (2'); no longer MP1.9 (2')
- net TR2: now also MP2.8 (2'); no longer MP2.9 (2')
- net TR3: now also MP3.8 (2'); no longer MP3.9 (2')
- net TR4: now also MP4.8 (2'); no longer MP4.9 (2')
- net VDDA: now also MP1.7 (1'), MP2.7 (1'), MP3.7 (1'), MP4.7 (1'); no longer MP1.8 (1'), MP2.8 (1'), MP3.8 (1'), MP4.8 (1')
Other:
- moved on the sheet: MP1A, MP2A, MP3A, MP4A
