File: FaderCtrl/HW/PCB/FaderCtrl/FaderCtrl.kicad_sch (KiCad schematic)
At the start: 110 parts, among them J1 UART, J10 MP4, J2 PDI, J3 PORTE, J4 VBAT, J5 Barrel_Jack_MountingPin, J6 PWM, J7 MP1, J8 MP2, J9 MP3, P1 USB_C_Plug_USB2.0, SW1 BTN1, SW2 BTN2, SW3 BTN3, U1 ATxmega256A3BU-A, U2 TSR_1-2450, U3 AMS1117-3.3, Y1 32k, Y2 12M

Commit message: layout progress on FaderCtrl
Parts:
- removed unit 4 of MP1
- removed unit 4 of MP2
- removed unit 4 of MP3
- removed unit 4 of MP4
- removed NT1: GNDD, NetTie:NetTie-2_SMD_Pad0.5mm, symbol Device:NetTie_2
- removed P1: USB_C_Plug_USB2.0, Connector_USB:USB_C_Receptacle_GCT_USB4125-xx-x-0190_6P_TopMnt_Horizontal, symbol Connector:USB_C_Plug_USB2.0
- removed R2: 56k, Resistor_SMD:R_0603_1608Metric_Pad0.98x0.95mm_HandSolder, symbol Device:R
- removed R3: 5k1, Resistor_SMD:R_0603_1608Metric_Pad0.98x0.95mm_HandSolder, symbol Device:R
- removed TP2: Vconn, TestPoint:TestPoint_Pad_D1.0mm, symbol Connector:TestPoint
- added J11: USB_B_Mini, Connector_USB:USB_Mini-B_Wuerth_65100516121_Horizontal, symbol Connector:USB_B_Mini
- added MPM1, MPM2, MPM3, MPM4: PSM01081A103B2_MotorOnly, Connector_JST:JST_XH_B2B-XH-A_1x02_P2.50mm_Vertical, symbol _MYLIBRARY:PSM01081A103B2_MotorOnly
- D2, D4, D6, D7: footprint Package_TO_SOT_SMD:SOT-323_SC-70 -> Package_TO_SOT_SMD:SOT-23_Handsoldering
- J5: symbol Connector:Barrel_Jack_MountingPin -> Connector:Barrel_Jack_Switch
- MP1, MP2, MP3, MP4: footprint footprints:PSM01-082A-103B2_MotorizedPot -> Connector_JST:JST_XH_B7B-XH-A_1x07_P2.50mm_Vertical; symbol _MYLIBRARY:PSM01081A103B2 -> _MYLIBRARY:PSM01081A103B2_PotOnly
- RV1, RV2, RV3, RV4: footprint PTL6015G0103B2_SlidePotLED -> footprints:PTL6015G0103B2_SlidePotLED
- TP4: footprint TestPoint:TestPoint_Pad_D1.0mm -> TestPoint:TestPoint_THTPad_D1.0mm_Drill0.5mm
- U4, U5: footprint HTSSOP-20-1EP_4.4x6.5mm_P0.65mm_EP3.4x6.5mm -> Package_SO:HTSSOP-20-1EP_4.4x6.5mm_P0.65mm_EP3.4x6.5mm
Connections:
- net GNDD is gone; now on net GND: C1.2, C13.2, C17.2, C2.2, C22.2, C26.2, C28.2, C29.2, C3.2, C32.2, C35.2, C36.2, C37.2, C38.2, C39.2, C4.2, D3.3 (K1), D3.4 (K2), D5.3 (K1), D5.4 (K2), J1.3 (Pin_3), J2.6 (Pin_6), J3.8 (Pin_8), J4.2 (Pin_2), J6.1 (Pin_1), NT2.1, SW1.1, SW2.1, SW3.1, U1.14 (GND), U1.24 (GND), U1.34 (GND), U1.44 (GND), U1.52 (GND), U1.60 (GND), U3.1 (GND), U4.20 (GND), U5.20 (GND), Y1.3
- net D+: now also J11.3 (D+)
- net D-: now also J11.2 (D-)
- net GND: now also J5.3, J11.5 (GND), J11.6 (Shield); no longer J5.MP (MountPin)
- net GNDA: now also MP1.7 (3'), MP2.7 (3'), MP3.7 (3'), MP4.7 (3'); no longer MP1.9 (3'), MP2.9 (3'), MP3.9 (3'), MP4.9 (3')
- net M1A: now also MPM1.1 (A); no longer MP1.1 (A)
- net M1B: now also MPM1.2 (B); no longer MP1.2 (B)
- net M2A: now also MPM2.1 (A); no longer MP2.1 (A)
- net M2B: now also MPM2.2 (B); no longer MP2.2 (B)
- net M3A: now also MPM3.1 (A); no longer MP3.1 (A)
- net M3B: now also MPM3.2 (B); no longer MP3.2 (B)
- net M4A: now also MPM4.1 (A); no longer MP4.1 (A)
- net M4B: now also MPM4.2 (B); no longer MP4.2 (B)
- net MP1N: now also MP4.3 (1); no longer MP4.5 (1)
- net MP1P: now also MP4.1 (3); no longer MP4.3
- net MP1S: now also MP4.2; no longer MP4.4 (2)
- net MP2N: now also MP3.3 (1); no longer MP3.5 (1)
- net MP2P: now also MP3.1 (3); no longer MP3.3
- net MP2S: now also MP3.2; no longer MP3.4 (2)
- net MP3N: now also MP2.3 (1); no longer MP2.5 (1)
- net MP3P: now also MP2.1 (3); no longer MP2.3
- net MP3S: now also MP2.2; no longer MP2.4 (2)
- net MP4N: now also MP1.3 (1); no longer MP1.5 (1)
- net MP4P: now also MP1.1 (3); no longer MP1.3
- net MP4S: now also MP1.2; no longer MP1.4 (2)
- net TP1: now also MP1.4 (T)
- net TP2: now also MP2.4 (T)
- net TP3: now also MP3.4 (T)
- net TP4: now also MP4.4 (T)
- net TR1: now also MP1.6 (2'); no longer MP1.8 (2')
- net TR2: now also MP2.6 (2'); no longer MP2.8 (2')
- net TR3: now also MP3.6 (2'); no longer MP3.8 (2')
- net TR4: now also MP4.6 (2'); no longer MP4.8 (2')
- net VBUS: now also J11.1 (VBUS)
- net VDDA: now also MP1.5 (1'), MP2.5 (1'), MP3.5 (1'), MP4.5 (1'); no longer MP1.7 (1'), MP2.7 (1'), MP3.7 (1'), MP4.7 (1')
- no-connect marks 2 -> 3
Other:
- moved on the sheet: J5

Commit message: layout fader done
Connections:
- net RXD: now also J1.2 (Pin_2); no longer J1.1 (Pin_1)
- net TXD: now also J1.1 (Pin_1); no longer J1.2 (Pin_2)
Other:
- moved on the sheet: J1

Commit message: dfgdggf
Parts:
- U4, U5: value ~ -> (none)
