File: FaderCtrl/HW/PCB/FaderCtrl/_autosave-FaderCtrl.kicad_sch (KiCad schematic)
At the start: 89 parts, among them J1 PDI, J2 Barrel_Jack_MountingPin, J3 PWM, J4 PORTD, J5 MPS, J6 MPP, J7 MPN, P1 USB_C_Plug_USB2.0, U1 ATxmega256A3BU-A, U2 TSR_1-2450, U3 AMS1117-3.3, Y1 32k

Commit message: a
Parts:
- added C40: 10n, Capacitor_SMD:C_0603_1608Metric_Pad1.08x0.95mm_HandSolder, symbol Device:C
- added SW1: SW_Push, symbol Switch:SW_Push
Connections:
- new net: C40.2, SW1.1
- new net: C40.1, SW1.2
Other:
- moved on the sheet: D2, D3, R2, R3, R6, R7

Commit message: a
Parts:
- removed J4: PORTD, symbol Connector_Generic:Conn_01x10
- added C17, C22: 10n, Capacitor_SMD:C_0603_1608Metric_Pad1.08x0.95mm_HandSolder, symbol Device:C
- added C2, C4: 10p, Capacitor_SMD:C_0603_1608Metric_Pad1.08x0.95mm_HandSolder, symbol Device:C
- added C45, C46: 100n, Capacitor_SMD:C_0603_1608Metric_Pad1.08x0.95mm_HandSolder, symbol Device:C
- added J1: UART, Connector_PinSocket_2.54mm:PinSocket_1x03_P2.54mm_Vertical, symbol Connector_Generic:Conn_01x03
- added J3: PORTE, Connector_PinSocket_1.27mm:PinSocket_1x08_P1.27mm_Vertical, symbol Connector_Generic:Conn_01x08
- added J4: VBAT, Connector_PinSocket_2.54mm:PinSocket_1x02_P2.54mm_Vertical, symbol Connector_Generic:Conn_01x02
- added R2: 56k, Resistor_SMD:R_0603_1608Metric_Pad0.98x0.95mm_HandSolder, symbol Device:R
- added R3: 5k1, Resistor_SMD:R_0603_1608Metric_Pad0.98x0.95mm_HandSolder, symbol Device:R
- added SW2: BTN2, footprints:SW_PUSH_6mm_2pins, symbol Switch:SW_Push
- added SW3: BTN3, footprints:SW_PUSH_6mm_2pins, symbol Switch:SW_Push
- added TP2: Vconn, TestPoint:TestPoint_Pad_D1.0mm, symbol Connector:TestPoint
- added TP3: TR1, TestPoint:TestPoint_THTPad_D1.0mm_Drill0.5mm, symbol Connector:TestPoint
- added TP4: ~{OE}, TestPoint:TestPoint_Pad_D1.0mm, symbol Connector:TestPoint
- added TP5: SLED1, TestPoint:TestPoint_Pad_D1.0mm, symbol Connector:TestPoint
- added TP8: SL1, TestPoint:TestPoint_THTPad_D1.0mm_Drill0.5mm, symbol Connector:TestPoint
- added Y2: 12M, Crystal:Crystal_SMD_HC49-SD, symbol Device:Crystal
- C1: now not fitted
- C3: renamed from C2; now not fitted
- D3: renamed from D2; footprint (none) -> LED_SMD:LED_Cree-PLCC4_3.2x2.8mm_CCW
- D5: renamed from D3; footprint (none) -> LED_SMD:LED_Cree-PLCC4_3.2x2.8mm_CCW
- J6: renamed from J3; footprint (none) -> Connector_PinSocket_1.27mm:PinSocket_1x09_P1.27mm_Vertical
- J7: renamed from J5; footprint (none) -> Connector_PinSocket_2.54mm:PinSocket_1x04_P2.54mm_Vertical
- J8: renamed from J6; footprint (none) -> Connector_PinSocket_2.54mm:PinSocket_1x04_P2.54mm_Vertical
- J9: renamed from J7; footprint (none) -> Connector_PinSocket_2.54mm:PinSocket_1x04_P2.54mm_Vertical
- JP1: value Jumper_3_Bridged12 -> Vin3v3
- JP2: value Jumper_2_Small_Bridged -> VDDA
- MP1, MP2, MP3, MP4: footprint Connector_PinSocket_2.54mm:PinSocket_1x09_P2.54mm_Vertical -> Connector_PinSocket_2.54mm:PinSocket_1x10_P2.54mm_Vertical
- NT1: value NetTie_2 -> GNDD
- NT2: value NetTie_2 -> GNDA
- SW1: value SW_Push -> BTN1; footprint (none) -> footprints:SW_PUSH_6mm_2pins
- TP9: renamed from TP4; footprint (none) -> TestPoint:TestPoint_THTPad_D1.0mm_Drill0.5mm
- U4, U5: footprint HTSSOP-20-1EP_4.4x6.5mm_P0.65mm_EP3.4x6.5mm -> Package_SO:HTSSOP-20-1EP_4.4x6.5mm_P0.65mm_EP3.4x6.5mm
- Y1: symbol Device:Crystal_GND2 -> Device:Crystal_GND3; now not fitted
- renumbered C8 to C10, C9 to C11, C10 to C12, C40 to C13, C11 to C14, C12 to C15, C13 to C16, C14 to C18, C16 to C19, C19 to C20, C15 to C21, C17 to C23, C18 to C24, C20 to C25, C21 to C26, C22 to C27, C23 to C28, C24 to C29, C25 to C30, C26 to C31, C27 to C32, C28 to C33, C29 to C34, C30 to C35, C31 to C36, C32 to C37, C33 to C38, C34 to C39, C35 to C40, C36 to C41, C37 to C42, C38 to C43, C39 to C44, C3 to C5, C4 to C6, C5 to C7, C6 to C8, C7 to C9, D4 to D2, D5 to D4, J1 to J2, J2 to J5, R6 to R10, R7 to R11, R10 to R12, R11 to R13, R8 to R6, R9 to R7, R2 to R8, R3 to R9, TP5 to TP10, TP6 to TP11, TP2 to TP6, TP3 to TP7
Connections:
- net BTN0 is gone; now on net BTN1: U1.11 (PB5)
- net PD0 is gone; now on net SLED1: U1.26 (PD0)
- net PD1 is gone; now on net SLED2: U1.27 (PD1)
- net PD2 is gone; now on net SLED3: U1.28 (PD2)
- net PD3 is gone; now on net SLED4: U1.29 (PD3)
- net PD4 is gone; now on net CP: U1.30 (PD4)
- net PD5 is gone; now on net ~{CP}: U1.31 (PD5)
- net PD6 is gone; now on net D-: U1.32 (PD6)
- net PD7 is gone; now on net D+: U1.33 (PD7)
- net +5V: no longer D2.1
- net BTN1: now also C13.1, SW1.2; no longer U1.12 (PB6)
- net BTN2: now also U1.12 (PB6), C17.1, SW2.2; no longer U1.13 (PB7)
- net CP: no longer U1.40 (PE4)
- net GNDA: now also C45.2, C46.2
- net GNDD: now also C13.2, SW1.1, Y1.3, C17.2, C2.2, C22.2, C4.2, J1.3 (Pin_3), J3.8 (Pin_8), J4.2 (Pin_2), R3.1, SW2.1, SW3.1; no longer Y1.2
- net SL1: now also TP8.1
- net SLED1: now also TP5.1; no longer U1.36 (PE0)
- net SLED2: no longer U1.37 (PE1)
- net SLED3: no longer U1.38 (PE2)
- net SLED4: no longer U1.39 (PE3)
- net TP3: now also U1.50 (PF4); no longer U1.48 (PF2)
- net TP4: now also U1.54 (PF6); no longer U1.49 (PF3)
- net TR1: now also TP3.1
- net VBUS: now also R2.2
- net VDD: now also J3.1 (Pin_1)
- net VDDA: now also C45.1, C46.1
- net Vdrive: now also D2.1
- net XTAL1: now also C2.1, Y2.1; no longer C3.1, Y1.3
- net XTAL2: now also C4.1, Y2.2; no longer C1.1, Y1.1
- net ~{CP}: no longer U1.41 (PE5)
- net ~{OE}: now also TP4.1
- net TOSC2: now reaches U1.42 (TOSC2)
- net TOSC2: now also C3.1, Y1.1
- net TOSC1: now reaches U1.43 (TOSC1)
- net TOSC1: now also C1.1, Y1.2
- net Vbat: now reaches U1.51 (VBAT)
- net Vbat: now also J4.1 (Pin_1)
- net CC: now reaches P1.A5 (CC)
- net CC: now also R2.1, R3.2
- net D+: now reaches P1.A6 (D+)
- net D-: now reaches P1.A7 (D-)
- net at P1.B5 (VCONN): now also TP2.1
- new net: J3.2 (Pin_2), U1.36 (PE0)
- new net: J3.3 (Pin_3), U1.37 (PE1)
- new net: J3.4 (Pin_4), U1.38 (PE2)
- new net: J3.5 (Pin_5), U1.39 (PE3)
- new net: J3.6 (Pin_6), U1.40 (PE4)
- new net: J3.7 (Pin_7), U1.41 (PE5)
- new net BTN3: C22.1, SW3.2, U1.13 (PB7)
- new net RXD: J1.1 (Pin_1), U1.48 (PF2)
- new net TXD: J1.2 (Pin_2), U1.49 (PF3)
- no-connect marks 4 -> 3
Other:
- company: (none) -> Xavier Bourlot
- title: (none) -> Fader Controller
- moved on the sheet: C42, C43, MP1D, MP2D, MP3D, MP4D, NT1, NT2, P1, TP1, TP10, TP11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
