File: FaderCtrl/HW/PCB/FaderCtrl/FaderCtrl.kicad_pcb (KiCad board)
At the start: 4 copper layers, 105 parts, among them J1 UART, J2 PDI, J3 PORTE, J4 VBAT, J5 Barrel_Jack_MountingPin, J6 PWM, J7 MPS, J8 MPP, J9 MPN, P1 USB_C_Plug_USB2.0, SW1 BTN1, SW2 BTN2, SW3 BTN3, U1 ATxmega256A3BU-A, U2 TSR_1-2450, U3 AMS1117-3.3, Y1 32k, Y2 12M

Commit message: a
Parts:
- TP1, TP10, TP11, TP3, TP4, TP5, TP6, TP7, TP8, TP9: moved to B.Cu
- moved C44 180.9 mm to (40.4, 169.5), turned to 180 degrees
- moved MP4 170.6 mm to (59.4, 172.0), turned to -90 degrees
- moved C46 163.8 mm to (40.4, 154.5), turned to 180 degrees
- moved MP3 151.8 mm to (59.4, 157.0), turned to -90 degrees
- moved C45 147.7 mm to (40.4, 139.5), turned to 180 degrees
- moved J9 137.7 mm to (74.6, 172.0), turned to -90 degrees
- moved J7 134.1 mm to (74.6, 169.4), turned to -90 degrees
- moved MP2 133.7 mm to (59.4, 142.0), turned to -90 degrees
- moved C41 133.0 mm to (40.4, 124.5), turned to 180 degrees
- moved J8 130.6 mm to (74.6, 167.0), turned to -90 degrees
- moved MP1 116.6 mm to (59.4, 127.0), turned to -90 degrees
- moved TP6 94.6 mm to (191.0, 81.0), turned to -90 degrees
- moved TP7 94.5 mm to (199.5, 81.0), turned to -90 degrees
- moved D2 94.4 mm to (195.5, 81.0), turned to 180 degrees
- moved C24 91.0 mm to (192.0, 83.5), turned to 180 degrees
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Routing:
- net VDD: track 0.00 -> 18.5 mm
- net GNDD: track 0.00 -> 9.91 mm, vias 0 -> 6
- net /TXD: track 0.00 -> 7.99 mm
- net /TOSC2: track 0.00 -> 6.38 mm
- net /TOSC1: track 0.00 -> 6.26 mm
- net /Vbat: track 0.00 -> 6.09 mm
- net /RXD: track 0.00 -> 5.96 mm
- net /SLED4: track 0.00 -> 5.89 mm
- net /SL1: track 0.00 -> 5.74 mm
- net /SLED3: track 0.00 -> 5.63 mm
- net /SLED2: track 0.00 -> 5.34 mm
- net /SLED1: track 0.00 -> 5.05 mm
- net /LED3: track 0.00 -> 4.78 mm, vias 0 -> 1
- net /SL2: track 0.00 -> 4.78 mm, vias 0 -> 1
- net /SL3: track 0.00 -> 4.40 mm, vias 0 -> 1
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
Commit message: a
Parts:
- added J10: MP4, Connector_PinHeader_2.54mm:PinHeader_1x03_P2.54mm_Vertical, F.Cu at (-4.00, 16.0)
- added RV1: PTL30-10R0-103B2, footprints:PTL6015G0103B2_SlidePotLED, F.Cu at (60.0, 0.00)
- added RV2: PTL30-10R0-103B2, footprints:PTL6015G0103B2_SlidePotLED, F.Cu at (75.0, 0.00)
- added RV3: PTL30-10R0-103B2, footprints:PTL6015G0103B2_SlidePotLED, F.Cu at (90.0, 0.00)
- added RV4: PTL30-10R0-103B2, footprints:PTL6015G0103B2_SlidePotLED, F.Cu at (105.0, 0.00)
- J7: value MPS -> MP1; footprint Connector_PinSocket_2.54mm:PinSocket_1x04_P2.54mm_Vertical -> Connector_PinHeader_2.54mm:PinHeader_1x03_P2.54mm_Vertical
- J8: value MPP -> MP2; footprint Connector_PinSocket_2.54mm:PinSocket_1x04_P2.54mm_Vertical -> Connector_PinHeader_2.54mm:PinHeader_1x03_P2.54mm_Vertical
- J9: value MPN -> MP3; footprint Connector_PinSocket_2.54mm:PinSocket_1x04_P2.54mm_Vertical -> Connector_PinHeader_2.54mm:PinHeader_1x03_P2.54mm_Vertical
- MP1, MP2, MP3, MP4: footprint Connector_PinSocket_2.54mm:PinSocket_1x10_P2.54mm_Vertical -> footprints:PSM01-082A-103B2_MotorizedPot
- moved J6 232.6 mm to (38.9, -78.0), turned to -90 degrees
- moved C18 231.0 mm to (-1.50, -34.5)
- moved C30 231.0 mm to (-4.50, -25.0)
- moved C33 231.0 mm to (-4.50, -21.5)
- moved C42 231.0 mm to (-4.50, -31.5)
- moved C5 231.0 mm to (-1.50, -32.5)
- moved TP10 231.0 mm to (-2.50, -30.0)
- moved TP4 231.0 mm to (1.50, -32.5)
- moved U4 231.0 mm to (0.31, -24.9)
- moved R4 224.5 mm to (24.8, -78.5), turned to -90 degrees
- moved C36 224.4 mm to (26.8, -77.5), turned to 90 degrees
- moved R5 223.7 mm to (23.3, -78.5), turned to -90 degrees
- moved R6 222.8 mm to (21.8, -78.5), turned to -90 degrees
- moved C38 222.2 mm to (38.0, -70.0), turned to 0 degrees
- moved R7 222.1 mm to (20.3, -78.5), turned to -90 degrees
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Connections:
- D2 pad 2: (no net) -> unconnected-(D2-Pad2)
- D4 pad 2: (no net) -> unconnected-(D4-Pad2)
- D6 pad 2: (no net) -> unconnected-(D6-Pad2)
- D7 pad 2: (no net) -> unconnected-(D7-Pad2)
- J7 pad 1: /MP1S -> /MP1P
- J7 pad 2: /MP2S -> /MP1S
- J7 pad 3: /MP3S -> /MP1N
- J8 pad 1: /MP1P -> /MP2P
- J8 pad 2: /MP2P -> /MP2S
- J8 pad 3: /MP3P -> /MP2N
- J9 pad 1: /MP1N -> /MP3P
- J9 pad 2: /MP2N -> /MP3S
- MP1 pad 3: (no net) -> /MP4P
- MP1 pad 4: /MP4P -> /MP4S
- MP1 pad 5: /MP4S -> /MP4N
- MP1 pad 6: /MP4N -> /TP1
- MP1 pad 7: /TP1 -> VDDA
- MP1 pad 8: VDDA -> /TR1
- MP1 pad 9: /TR1 -> GNDA
- MP2 pad 3: (no net) -> /MP3P
- MP2 pad 4: /MP3P -> /MP3S
- MP2 pad 5: /MP3S -> /MP3N
- MP2 pad 6: /MP3N -> /TP2
- MP2 pad 7: /TP2 -> VDDA
- MP2 pad 8: VDDA -> /TR2
- MP2 pad 9: /TR2 -> GNDA
- MP3 pad 3: (no net) -> /MP2P
- MP3 pad 4: /MP2P -> /MP2S
- MP3 pad 5: /MP2S -> /MP2N
- MP3 pad 6: /MP2N -> /TP3
- MP3 pad 7: /TP3 -> VDDA
- MP3 pad 8: VDDA -> /TR3
- MP3 pad 9: /TR3 -> GNDA
- MP4 pad 3: (no net) -> /MP1P
- MP4 pad 4: /MP1P -> /MP1S
- MP4 pad 5: /MP1S -> /MP1N
- MP4 pad 6: /MP1N -> /TP4
- MP4 pad 7: /TP4 -> VDDA
- MP4 pad 8: VDDA -> /TR4
- MP4 pad 9: /TR4 -> GNDA
- U1 pad 10: /~{OE} -> /SL1
- U1 pad 11: /BTN1 -> /SL2
- U1 pad 12: /BTN2 -> /SL3
- U1 pad 13: /BTN3 -> /SL4
- U1 pad 2: /SL1 -> /LED0
- U1 pad 3: /SL2 -> /LED1
- U1 pad 4: /SL3 -> /LED2
- U1 pad 5: /SL4 -> /LED3
- U1 pad 55: unconnected-(U1-PF7-Pad55) -> /~{OE}
- U1 pad 6: /LED0 -> VDDA
- U1 pad 7: /LED1 -> /BTN1
- U1 pad 8: /LED2 -> /BTN2
- U1 pad 9: /LED3 -> /BTN3
- U4 pad 21: (no net) -> GND
- U5 pad 21: (no net) -> GND
Other:
- board outline added: 123 x 100 mm
